Commit message: URDF update

File: motoman_sda10f_support/urdf/aruco_marker_macro.xacro (robot description, xacro)
@@ -2,4 +2,5 @@
 <robot xmlns:xacro="http://ros.org/wiki/xacro">
   <xacro:macro name="aruco_marker" params="prefix"><!-- Attach aruco marker  -->
+  </xacro:macro>
   <link name="aruco_marker_link">
       <inertial>
@@ -23,8 +24,31 @@
     </link>
   <joint name="aruco_marker_joint" type="fixed">
-    <origin xyz="${0.144-0.045+0.045} ${-0.045+0.045} -0.00" rpy="0 0 0" />
+    <origin xyz="${0.144-0.045+0.045} ${-0.045+0.045} -0.00" rpy="1.57 0 0" />
     <parent link="robotiq_85_base_link"/>
     <child link="aruco_marker_link"/>
   </joint>
-  </xacro:macro>
 </robot>
+ <!-- <link name="aruco_marker_link">
+      <inertial>
+        <origin xyz="0.01747 0.0014 0.128" rpy="0 0 0" />
+        <mass value="0.01" />
+        <inertia ixx="0.1"  ixy="0"  ixz="0" iyy="0.1" iyz="0" izz="0.1" />
+      </inertial>
+      <visual>
+        <geometry>
+          <mesh filename="package://motoman_sda10f_support/meshes/environment/marker582_8cm.dae"/>
+        </geometry>
+        <material name="DarkGrey" />
+      </visual>
+      <collision>
+        <origin xyz="0 0 0" rpy="0 0 0" />
+        <geometry>
+	         <box size="0.09 0.09 0.0001"/>
+        </geometry>
+      </collision>
+    </link>
+  <joint name="aruco_marker_joint" type="fixed">
+    <origin xyz="${0.144-0.045} -0.045 0.00" rpy="0 0 0" />
+    <parent link="robotiq_85_base_link"/>
+    <child link="aruco_marker_link"/>
+  </joint>>-->

Commit message: aruco_correction

File: motoman_sda10f_support/urdf/aruco_marker_macro.xacro (robot description, xacro)
@@ -10,5 +10,5 @@
       </inertial>
       <visual>
-        <origin xyz="-0.045 -0.045 0" rpy="0 0 0" />
+        <origin xyz="-0.045 0 0.045" rpy="-1.57 0 0" />
         <geometry>
           <mesh filename="package://motoman_sda10f_support/meshes/environment/marker582_8cm.dae"/>
@@ -29,26 +29,2 @@
   </joint>
 </robot>
- <!-- <link name="aruco_marker_link">
-      <inertial>
-        <origin xyz="0.01747 0.0014 0.128" rpy="0 0 0" />
-        <mass value="0.01" />
-        <inertia ixx="0.1"  ixy="0"  ixz="0" iyy="0.1" iyz="0" izz="0.1" />
-      </inertial>
-      <visual>
-        <geometry>
-          <mesh filename="package://motoman_sda10f_support/meshes/environment/marker582_8cm.dae"/>
-        </geometry>
-        <material name="DarkGrey" />
-      </visual>
-      <collision>
-        <origin xyz="0 0 0" rpy="0 0 0" />
-        <geometry>
-	         <box size="0.09 0.09 0.0001"/>
-        </geometry>
-      </collision>
-    </link>
-  <joint name="aruco_marker_joint" type="fixed">
-    <origin xyz="${0.144-0.045} -0.045 0.00" rpy="0 0 0" />
-    <parent link="robotiq_85_base_link"/>
-    <child link="aruco_marker_link"/>
-  </joint>>-->

Commit message: Package URDF modifications

File: motoman_sda10f_support/urdf/aruco_marker_macro.xacro (robot description, xacro)
@@ -10,5 +10,5 @@
       </inertial>
       <visual>
-        <origin xyz="-0.045 0 0.045" rpy="-1.57 0 0" />
+        <origin xyz="-0.045 0 0.045" rpy="0 0 0" />
         <geometry>
           <mesh filename="package://motoman_sda10f_support/meshes/environment/marker582_8cm.dae"/>
@@ -24,5 +24,5 @@
     </link>
   <joint name="aruco_marker_joint" type="fixed">
-    <origin xyz="${0.144-0.045+0.045} ${-0.045+0.045} -0.00" rpy="1.57 0 0" />
+    <origin xyz="0.18 0 0" rpy="0 0 3.1416" />
     <parent link="robotiq_85_base_link"/>
     <child link="aruco_marker_link"/>

File: motoman_sda10f_support/urdf/sda10f_macro.xacro (robot description, xacro)
@@ -19,9 +19,9 @@
 		<xacro:robotiq_c2_model prefix=""/>
 		<xacro:s-model_articulated prefix=""/>
-		<!--Grippers with robotr joints-->
+		<!--Grippers with robot joints-->
 		<joint name="left_gripper_to_robot" type="fixed">
 			<parent link="${prefix}arm_left_link_tool0" />
 			<child link = "${prefix}robotiq_85_adapter_link" />
-			<origin xyz="0 0 0" rpy="0 1.5708 2.3562" />
+			<origin xyz="0 0 0" rpy="0 1.5708 2.3562" /> <!--PLATINA -0.035 -->
 		</joint>
 		<joint name="right_gripper_to_robot" type="fixed">
@@ -36,11 +36,12 @@
 		<joint name="arm_right_tool0_to_tcp" type="fixed" >
 			<parent link="${prefix}arm_right_link_tool0" />
-			<child link = "${prefix}arm_right_tcp_link" />
-			<origin xyz="0 0 -0.16" rpy="3.1416 0 0" />
+			<child link ="${prefix}arm_right_tcp_link" />
+			<origin xyz="0 0 -0.23" rpy="3.1416 0 0" />
 		</joint>
+		<!--TCPs defined in teach pendant-->
 		<joint name="arm_left_tool0_to_tcp" type="fixed" >
 			<parent link="${prefix}arm_left_link_tool0" />
 			<child link = "${prefix}arm_left_tcp_link" />
-			<origin xyz="0 0 -0.12" rpy="3.1416 0 0.7854" />
+			<origin xyz="0 0 -0.15" rpy="3.1416 0 0.7854" />
 		</joint>
 		</xacro:macro>

File: motoman_sda10f_support/urdf/simple_sda10f_macro.xacro (robot description, xacro)
@@ -3,8 +3,9 @@
      <xacro:include filename="$(find motoman_sda10f_support)/urdf/common_torso_macro.xacro" />
      <xacro:include filename="$(find motoman_sda10f_support)/urdf/arm_macro.xacro" />
-     <xacro:include filename="$(find motoman_sda10f_support)/urdf/aruco_marker_macro.xacro"/>
      <xacro:include filename="$(find robotiq_c2_model_visualization)/urdf/robotiq_c2_model_macro.xacro"/>
+     <xacro:include filename="$(find robotiq_s_model_visualization)/cfg/s-model_articulated_macro.xacro"/>
      <xacro:include filename="$(find motoman_sda10f_support)/urdf/kinect_macro.xacro" />
-	<xacro:include filename="$(find motoman_sda10f_support)/urdf/simple_environment_macro.xacro"/>
+	<xacro:include filename="$(find motoman_sda10f_support)/urdf/environment_macro.xacro"/>
+	<xacro:include filename="$(find motoman_sda10f_support)/urdf/aruco_marker_macro.xacro"/>
      <xacro:macro name="motoman_sda10f" params="prefix">
         <xacro:torso name="${prefix}torso" prefix="${prefix}torso_"/>
@@ -16,8 +17,29 @@
         </xacro:motoman_arm>
         <xacro:robotiq_c2_model prefix=""/>
-        	<joint name="left_gripper_to_robot" type="fixed">
+		<xacro:s-model_articulated prefix=""/>
+		<!--Grippers with robot joints-->
+		<joint name="left_gripper_to_robot" type="fixed">
 			<parent link="${prefix}arm_left_link_tool0" />
 			<child link = "${prefix}robotiq_85_adapter_link" />
 			<origin xyz="0 0 0" rpy="0 1.5708 2.3562" />
+		</joint>
+		<joint name="right_gripper_to_robot" type="fixed">
+			<parent link="${prefix}arm_right_link_tool0" />
+			<child link = "${prefix}palm" />
+			<origin xyz="0 0 0" rpy="-1.5708 0 1.5708" />
+		</joint>
+		<!--Create and update TCP pose -->
+		<link name="arm_right_tcp_link" />
+		<link name="arm_left_tcp_link" />
+		<!--Define the position of the TCP with respect to the arm flange-->
+		<joint name="arm_right_tool0_to_tcp" type="fixed" >
+			<parent link="${prefix}arm_right_link_tool0" />
+			<child link = "${prefix}arm_right_tcp_link" />
+			<origin xyz="0 0 -0.16" rpy="3.1416 0 0" />
+		</joint>
+		<joint name="arm_left_tool0_to_tcp" type="fixed" >
+			<parent link="${prefix}arm_left_link_tool0" />
+			<child link = "${prefix}arm_left_tcp_link" />
+			<origin xyz="0 0 -0.12" rpy="3.1416 0 0.7854" />
 		</joint>
      </xacro:macro>

Commit message: URDF and launch files corrections

File: motoman_sda10f_support/urdf/aruco_marker_macro.xacro (robot description, xacro)
@@ -23,7 +23,14 @@
       </collision>
     </link>
-  <joint name="aruco_marker_joint" type="fixed">
+    <!--Left arm-->
+  <!--joint name="aruco_marker_joint" type="fixed">
     <origin xyz="0.18 0 0" rpy="0 0 3.1416" />
     <parent link="robotiq_85_base_link"/>
+    <child link="aruco_marker_link"/>
+  </joint-->
+   <!--Right arm -->
+    <joint name="aruco_marker_joint" type="fixed">
+    <origin xyz="0 0 0.1425" rpy="0 -1.5708 -1.5708" />
+    <parent link="arm_right_tcp_link"/>
     <child link="aruco_marker_link"/>
   </joint>

File: motoman_sda10f_support/urdf/environment_macro.xacro (robot description, xacro)
@@ -14,4 +14,22 @@
 				<!--color rgba="${240/255} ${240/255} ${240/255} 1"/-->
 			</material>
+		</visual>
+</link>
+	<link name="arm_left_gripper_support">
+		<visual>
+			<geometry>
+				<cylinder length="0.024" radius="0.0405"/>
+			</geometry>
+			<origin xyz="0 0 0"/>
+			<material name="gray_conveyor"/>
+		</visual>
+</link>
+	<link name="arm_right_gripper_support">
+		<visual>
+			<geometry>
+				<cylinder length="0.01" radius="0.04"/>
+			</geometry>
+			<origin xyz="0 0 0"/>
+			<material name="gray_conveyor"/>
 		</visual>
 </link>
@@ -114,4 +132,14 @@
 		<origin xyz="0.572 -1.244 -0.252" rpy="0 0 -1.571"/>
 	</joint>
+	<joint name="arm_left_gripper_support_to_robot" type="fixed">
+		<parent link="arm_left_link_tool0"/>
+		<child link="arm_left_gripper_support"/>
+		<origin xyz="0 0 -0.022" rpy="0 0 0"/>
+	</joint>
+	<joint name="arm_right_gripper_support_to_robot" type="fixed">
+		<parent link="arm_right_link_tool0"/>
+		<child link="arm_right_gripper_support"/>
+		<origin xyz="0 0 -0.015" rpy="0 0 0"/>
+	</joint>
 	<joint name="feeder_table_to_robot" type="fixed">
 		<parent link="torso_base_link"/>

File: motoman_sda10f_support/urdf/sda10f_macro.xacro (robot description, xacro)
@@ -3,5 +3,5 @@
 	<xacro:include filename="$(find motoman_sda10f_support)/urdf/common_torso_macro.xacro" />
 	<xacro:include filename="$(find motoman_sda10f_support)/urdf/arm_macro.xacro" />
-	<xacro:include filename="$(find robotiq_c2_model_visualization)/urdf/robotiq_c2_model_macro.xacro"/>
+	<xacro:include filename="$(find motoman_sda10f_support)/urdf/robotiq_c2_model_macro.xacro"/>
 	<xacro:include filename="$(find robotiq_s_model_visualization)/cfg/s-model_articulated_macro.xacro"/>
 	<xacro:include filename="$(find motoman_sda10f_support)/urdf/kinect_macro.xacro" />
@@ -22,11 +22,11 @@
 		<joint name="left_gripper_to_robot" type="fixed">
 			<parent link="${prefix}arm_left_link_tool0" />
-			<child link = "${prefix}robotiq_85_adapter_link" />
-			<origin xyz="0 0 0" rpy="0 1.5708 2.3562" /> <!--PLATINA -0.035 -->
+			<child link = "${prefix}robotiq_85_base_link" />
+			<origin xyz="0 0 -0.034" rpy="0 1.5708 2.3562" />
 		</joint>
 		<joint name="right_gripper_to_robot" type="fixed">
 			<parent link="${prefix}arm_right_link_tool0" />
 			<child link = "${prefix}palm" />
-			<origin xyz="0 0 0" rpy="-1.5708 0 1.5708" />
+			<origin xyz="0 0 -0.065" rpy="-1.5708 0 1.5708" />
 		</joint>
 		<!--Create and update TCP pose -->
@@ -36,8 +36,7 @@
 		<joint name="arm_right_tool0_to_tcp" type="fixed" >
 			<parent link="${prefix}arm_right_link_tool0" />
-			<child link ="${prefix}arm_right_tcp_link" />
+			<child link = "${prefix}arm_right_tcp_link" />
 			<origin xyz="0 0 -0.23" rpy="3.1416 0 0" />
 		</joint>
-		<!--TCPs defined in teach pendant-->
 		<joint name="arm_left_tool0_to_tcp" type="fixed" >
 			<parent link="${prefix}arm_left_link_tool0" />

File: motoman_sda10f_support/urdf/simple_sda10f_macro.xacro (robot description, xacro)
@@ -3,5 +3,5 @@
      <xacro:include filename="$(find motoman_sda10f_support)/urdf/common_torso_macro.xacro" />
      <xacro:include filename="$(find motoman_sda10f_support)/urdf/arm_macro.xacro" />
-     <xacro:include filename="$(find robotiq_c2_model_visualization)/urdf/robotiq_c2_model_macro.xacro"/>
+     <xacro:include filename="$(find motoman_sda10f_support)/urdf/robotiq_c2_model_macro.xacro"/>
      <xacro:include filename="$(find robotiq_s_model_visualization)/cfg/s-model_articulated_macro.xacro"/>
      <xacro:include filename="$(find motoman_sda10f_support)/urdf/kinect_macro.xacro" />
@@ -21,11 +21,11 @@
 		<joint name="left_gripper_to_robot" type="fixed">
 			<parent link="${prefix}arm_left_link_tool0" />
-			<child link = "${prefix}robotiq_85_adapter_link" />
-			<origin xyz="0 0 0" rpy="0 1.5708 2.3562" />
+			<child link = "${prefix}robotiq_85_base_link" />
+			<origin xyz="0 0 -0.034" rpy="0 1.5708 2.3562" />
 		</joint>
 		<joint name="right_gripper_to_robot" type="fixed">
 			<parent link="${prefix}arm_right_link_tool0" />
 			<child link = "${prefix}palm" />
-			<origin xyz="0 0 0" rpy="-1.5708 0 1.5708" />
+			<origin xyz="0 0 -0.065" rpy="-1.5708 0 1.5708" />
 		</joint>
 		<!--Create and update TCP pose -->
@@ -36,10 +36,10 @@
 			<parent link="${prefix}arm_right_link_tool0" />
 			<child link = "${prefix}arm_right_tcp_link" />
-			<origin xyz="0 0 -0.16" rpy="3.1416 0 0" />
+			<origin xyz="0 0 -0.23" rpy="3.1416 0 0" />
 		</joint>
 		<joint name="arm_left_tool0_to_tcp" type="fixed" >
 			<parent link="${prefix}arm_left_link_tool0" />
 			<child link = "${prefix}arm_left_tcp_link" />
-			<origin xyz="0 0 -0.12" rpy="3.1416 0 0.7854" />
+			<origin xyz="0 0 -0.15" rpy="3.1416 0 0.7854" />
 		</joint>
      </xacro:macro>
