Commit message: urdf changes

File: motoman_sda10f_support/urdf/environment_macro.xacro (robot description, xacro)
@@ -160,5 +160,5 @@
 		<parent link="table"/>
 		<child link="worktable"/>
-		<origin xyz="0 1.28 -0.76" rpy="0 0 0"/> <!--Accurate 1.274 aprox 1.28-->
+		<origin xyz="0 1.28 -0.76" rpy="0 0 0"/>
 	</joint>
 	<joint name="beacon_to_robot" type="fixed">

File: motoman_sda10f_support/urdf/sda10f_macro.xacro (robot description, xacro)
@@ -8,4 +8,5 @@
 	<xacro:include filename="$(find motoman_sda10f_support)/urdf/environment_macro.xacro"/>
 	<xacro:include filename="$(find motoman_sda10f_support)/urdf/visual_environment_macro.xacro"/>
+	<xacro:include filename="$(find motoman_sda10f_support)/urdf/real_sense_macro.xacro"/>
 		<xacro:macro name="motoman_sda10f" params="prefix">
 		<xacro:torso name="${prefix}torso" prefix="${prefix}torso_"/>

File: motoman_sda10f_support/urdf/simple_sda10f_macro.xacro (robot description, xacro)
@@ -7,5 +7,6 @@
      <xacro:include filename="$(find motoman_sda10f_support)/urdf/kinect_macro.xacro" />
 	<xacro:include filename="$(find motoman_sda10f_support)/urdf/environment_macro.xacro"/>
-	<xacro:include filename="$(find motoman_sda10f_support)/urdf/aruco_marker_macro.xacro"/>
+	<xacro:include filename="$(find motoman_sda10f_support)/urdf/real_sense_macro.xacro"/>
+	<!--xacro:include filename="$(find motoman_sda10f_support)/urdf/aruco_marker_macro.xacro"/-->
      <xacro:macro name="motoman_sda10f" params="prefix">
         <xacro:torso name="${prefix}torso" prefix="${prefix}torso_"/>

Commit message: new wait poses added

File: motoman_sda10f_support/urdf/environment_macro.xacro (robot description, xacro)
@@ -155,5 +155,5 @@
 		<parent link="torso_base_link"/>
 		<child link="table"/>
-		<origin xyz="0.7 0 -0.3" rpy="1.571 0 -1.571"/>
+		<origin xyz="0.7 0 -0.34" rpy="1.571 0 -1.571"/> <!--MODIFIED BY NICOLAS TODO-->
 	</joint>
 	<joint name="worktable_to_robot" type="fixed">

Commit message: New poses added

File: motoman_sda10f_support/urdf/environment_macro.xacro (robot description, xacro)
@@ -97,5 +97,5 @@
 		</visual>
 </link-->
-	<link name="mps">
+	<!--link name="mps">
 		<visual>
 			<geometry>
@@ -113,6 +113,6 @@
 				<origin xyz= "-0.7 0 -1.40"/>
 		</collision>
-</link>
-	<!--link name="MPS_FAKE">
+</link-->
+	<link name="MPS_FAKE">
 		<visual>
 			<geometry>
@@ -124,5 +124,5 @@
 			</material>
 		</visual>
-</link-->
+</link>
 		<!-- joint list -->
 	<joint name="coveyor_to_robot" type="fixed">
@@ -172,14 +172,14 @@
 		<origin xyz="-0.53 -0.54 -0.3" rpy="1.571 0 1.571"/>
 	</joint-->
-		<joint name="mps_to_robot" type="fixed">
+		<!--joint name="mps_to_robot" type="fixed">
 		<parent link="torso_base_link"/>
 		<child link="mps"/>
-		<origin xyz="-0.111 -1.405 -0.3" rpy="1.571 0 1.571"/> <!--Sumo 5cm a las MPS por si acaso-->
-	</joint>
-		<!--joint name="MPS_FAKE_to_robot" type="fixed">
+		<origin xyz="-0.111 -1.405 -0.3" rpy="1.571 0 1.571"/--> <!--Sumo 5cm a las MPS por si acaso-->
+	<!--/joint-->
+		<joint name="MPS_FAKE_to_robot" type="fixed">
 		<parent link="torso_base_link"/>
 		<child link="MPS_FAKE"/>
-		<origin xyz="-1.35 0.6 -0.3" rpy="0 0 -1.5708"/--> <!--Sumo 5cm a las MPS por si acaso-->
-	<!--/joint-->
+		<origin xyz="-1.35 0.6 -0.3" rpy="0 0 -1.5708"/> <!--Sumo 5cm a las MPS por si acaso-->
+	</joint>
 		<!-- end of joint list -->
 	</xacro:macro>

Commit message: se adciono el nuevo gripper , tambien se coloco la mesa de herramientas

File: motoman_sda10f_support/urdf/environment_macro.xacro (robot description, xacro)
@@ -1,5 +1,7 @@
 <?xml version="1.0" ?>
 <model xmlns:xacro="http://ros.org/wiki/xacro">
+	<xacro:include filename="$(find motoman_sda10f_support)/urdf/zed_macro.xacro"/><!-- ZED camera -->
 	<xacro:macro name="environment" params="name prefix">
+	<xacro:zed_camera prefix=""/>
 		<!-- link list -->
 	<link name="conveyor">
@@ -16,8 +18,8 @@
 		</visual>
 </link>
-	<link name="arm_left_gripper_support">
-		<visual>
-			<geometry>
-				<cylinder length="0.024" radius="0.0405"/>
+	<link name="arm_right_gripper_support">
+		<visual>
+			<geometry>
+				<cylinder length="0.01" radius="0.04"/>
 			</geometry>
 			<origin xyz="0 0 0"/>
@@ -25,8 +27,8 @@
 		</visual>
 </link>
-	<link name="arm_right_gripper_support">
-		<visual>
-			<geometry>
-				<cylinder length="0.01" radius="0.04"/>
+	<link name="feeder_table">
+		<visual>
+			<geometry>
+				<mesh filename="package://motoman_sda10f_support/meshes/environment/feeder_table.stl" scale="0.01 0.01 0.01"/>
 			</geometry>
 			<origin xyz="0 0 0"/>
@@ -34,5 +36,5 @@
 		</visual>
 </link>
-	<link name="feeder_table">
+	<link name="feeder_table_2">
 		<visual>
 			<geometry>
@@ -43,14 +45,5 @@
 		</visual>
 </link>
-	<link name="feeder_table_2">
-		<visual>
-			<geometry>
-				<mesh filename="package://motoman_sda10f_support/meshes/environment/feeder_table.stl" scale="0.01 0.01 0.01"/>
-			</geometry>
-			<origin xyz="0 0 0"/>
-			<material name="gray_conveyor"/>
-		</visual>
-</link>
-	<link name="table">
+	<!--link name="table">
 		<visual>
 			<geometry>
@@ -63,6 +56,6 @@
 			</material>
 		</visual>
-</link>
-	<link name="worktable">
+</link-->
+	<!--link name="worktable">
 		<visual>
 			<geometry>
@@ -72,4 +65,15 @@
 			<material name="gray_worktable">
 				<color rgba="${45/255} ${135/255} ${149/255} 1"/>
+			</material>
+		</visual>
+</link-->
+	<link name="worktable">
+		<visual>
+			<geometry>
+				<mesh filename="package://motoman_sda10f_support/meshes/environment/table_new.stl" scale="0.001 0.001 0.001"/>
+			</geometry>
+			<origin xyz="0 0 0"/>
+			<material name="gray_conveyor">
+				<texture filename="package://motoman_sda10f_support/meshes/environment/textures/red.png"/>
 			</material>
 		</visual>
@@ -114,5 +118,5 @@
 		</collision>
 </link-->
-	<link name="MPS_FAKE">
+	<!--link name="MPS_FAKE">
 		<visual>
 			<geometry>
@@ -122,4 +126,15 @@
 			<material name="cyan_mps">
 				<color rgba="${168/255} ${224/255} ${198/255} 1"/>
+			</material>
+		</visual>
+</link-->
+	<link name="tool_table">
+		<visual>
+			<geometry>
+				<mesh filename="package://motoman_sda10f_support/meshes/environment/tool_table.STL"/>
+			</geometry>
+			<origin xyz="0 0 0"/>
+			<material name="gray_conveyor">
+				<texture filename="package://motoman_sda10f_support/meshes/environment/textures/red.png"/>
 			</material>
 		</visual>
@@ -131,9 +146,4 @@
 		<!--origin xyz="-2.92 -2.45 0.13" rpy="0 0 -1.571" OJO 0.618 PARA LA BANDA ORIGINAL/-->
 		<origin xyz="0.572 -1.244 -0.252" rpy="0 0 -1.571"/>
-	</joint>
-	<joint name="arm_left_gripper_support_to_robot" type="fixed">
-		<parent link="arm_left_link_tool0"/>
-		<child link="arm_left_gripper_support"/>
-		<origin xyz="0 0 -0.022" rpy="0 0 0"/>
 	</joint>
 	<joint name="arm_right_gripper_support_to_robot" type="fixed">
@@ -152,13 +162,18 @@
 		<origin xyz="1.11 0 0" rpy="0 0 0"/>
 	</joint>
-	<joint name="table_to_robot" type="fixed">
+	<!--joint name="table_to_robot" type="fixed">
 		<parent link="torso_base_link"/>
 		<child link="table"/>
-		<origin xyz="0.7 0 -0.34" rpy="1.571 0 -1.571"/> <!--MODIFIED BY NICOLAS TODO-->
-	</joint>
-	<joint name="worktable_to_robot" type="fixed">
+		<origin xyz="0.7 0 -0.34" rpy="1.571 0 -1.571"/>
+	</joint-->
+	<!--joint name="worktable_to_robot" type="fixed">
 		<parent link="table"/>
 		<child link="worktable"/>
 		<origin xyz="0 1.28 -0.76" rpy="0 0 0"/>
+	</joint-->
+	<joint name="worktable_to_robot" type="fixed">
+		<parent link="torso_base_link"/>
+		<child link="worktable"/>
+		<origin xyz="0.52 0 0.29" rpy="0 0  1.57"/>
 	</joint>
 	<joint name="beacon_to_robot" type="fixed">
@@ -177,8 +192,19 @@
 		<origin xyz="-0.111 -1.405 -0.3" rpy="1.571 0 1.571"/--> <!--Sumo 5cm a las MPS por si acaso-->
 	<!--/joint-->
-		<joint name="MPS_FAKE_to_robot" type="fixed">
+	<!--joint name="MPS_FAKE_to_robot" type="fixed">
 		<parent link="torso_base_link"/>
 		<child link="MPS_FAKE"/>
-		<origin xyz="-1.35 0.6 -0.3" rpy="0 0 -1.5708"/> <!--Sumo 5cm a las MPS por si acaso-->
+		<origin xyz="-1.35 0.6 -0.3" rpy="0 0 -1.5708"/> <!Sumo 5cm a las MPS por si acaso-->
+	<!--/joint-->
+	<!-- Camera zed -->
+	<joint name="zed_camera" type="fixed">
+		<parent link="torso_base_link" />
+		<child link = "zed_camera_center" />
+		<origin xyz="0.8 0.05 2.05" rpy="0 1.57 0" />
+	</joint>
+	<joint name="tooltable_to_robot" type="fixed">
+		<parent link="conveyor"/>
+		<child link="tool_table"/>
+		<origin xyz="-1.8 -1.33 0.68" rpy="1.57 0 3.14"/>
 	</joint>
 		<!-- end of joint list -->

File: motoman_sda10f_support/urdf/sda10f_macro.xacro (robot description, xacro)
@@ -1,29 +1,24 @@
 <?xml version="1.0" ?>
 <robot xmlns:xacro="http://ros.org/wiki/xacro">
-	<xacro:include filename="$(find motoman_sda10f_support)/urdf/common_torso_macro.xacro" />
-	<xacro:include filename="$(find motoman_sda10f_support)/urdf/arm_macro.xacro" />
-	<xacro:include filename="$(find motoman_sda10f_support)/urdf/robotiq_c2_model_macro.xacro"/>
-	<xacro:include filename="$(find robotiq_s_model_visualization)/cfg/s-model_articulated_macro.xacro"/>
-	<xacro:include filename="$(find motoman_sda10f_support)/urdf/kinect_macro.xacro" />
+     <xacro:include filename="$(find motoman_sda10f_support)/urdf/common_torso_macro.xacro" />
+     <xacro:include filename="$(find motoman_sda10f_support)/urdf/arm_macro.xacro" />
+     <xacro:include filename="$(find robotiq_s_model_visualization)/cfg/s-model_articulated_macro.xacro"/>
+     <xacro:include filename="$(find motoman_sda10f_support)/urdf/kinect_macro.xacro" />
 	<xacro:include filename="$(find motoman_sda10f_support)/urdf/environment_macro.xacro"/>
-	<xacro:include filename="$(find motoman_sda10f_support)/urdf/visual_environment_macro.xacro"/>
 	<xacro:include filename="$(find motoman_sda10f_support)/urdf/real_sense_macro.xacro"/>
-		<xacro:macro name="motoman_sda10f" params="prefix">
-		<xacro:torso name="${prefix}torso" prefix="${prefix}torso_"/>
-		<xacro:motoman_arm name="${prefix}arm_left" prefix="${prefix}arm_left_" parent="${prefix}torso_link_b1" reflect="1">
-			<origin xyz="0.09996 0.0275 0.32214" rpy="1.57 0 0" />
-		</xacro:motoman_arm>
-		<xacro:motoman_arm name="${prefix}arm_right" prefix="${prefix}arm_right_" parent="${prefix}torso_link_b1" reflect="-1">
-			<origin xyz="0.09996 -0.0275 0.32214" rpy="1.57 0 0" />
-		</xacro:motoman_arm>
-		<!--Grippers-->
-		<xacro:robotiq_c2_model prefix=""/>
+	<!--xacro:include filename="$(find motoman_sda10f_support)/urdf/zed_macro.xacro"/--><!-- ZED camera LLAMADA EN ENVIRONMENT.XACRO OJOOOOO MODIFICAR ESTO-->
+	<!--xacro:include filename="$(find motoman_sda10f_support)/urdf/aruco_marker_macro.xacro"/-->
+        <xacro:include filename="$(find robotiq_85_description)/urdf/robotiq_85_gripper.xacro" />
+     <xacro:macro name="motoman_sda10f" params="prefix">
+        <xacro:torso name="${prefix}torso" prefix="${prefix}torso_"/>
+        <xacro:motoman_arm name="${prefix}arm_left" prefix="${prefix}arm_left_" parent="${prefix}torso_link_b1" reflect="1">
+            <origin xyz="0.09996 0.0275 0.32214" rpy="1.57 0 0" />
+        </xacro:motoman_arm>
+        <xacro:motoman_arm name="${prefix}arm_right" prefix="${prefix}arm_right_" parent="${prefix}torso_link_b1" reflect="-1">
+            <origin xyz="0.09996 -0.0275 0.32214" rpy="1.57 0 0" />
+        </xacro:motoman_arm>
+        <!--xacro:robotiq_c2_model prefix=""/-->
 		<xacro:s-model_articulated prefix=""/>
 		<!--Grippers with robot joints-->
-		<joint name="left_gripper_to_robot" type="fixed">
-			<parent link="${prefix}arm_left_link_tool0" />
-			<child link = "${prefix}robotiq_85_base_link" />
-			<origin xyz="0 0 -0.034" rpy="0 1.5708 2.3562" />
-		</joint>
 		<joint name="right_gripper_to_robot" type="fixed">
 			<parent link="${prefix}arm_right_link_tool0" />
@@ -34,4 +29,7 @@
 		<link name="arm_right_tcp_link" />
 		<link name="arm_left_tcp_link" />
+		<xacro:robotiq_85_gripper prefix="" parent="arm_left_link_tool0" >
+        		<origin xyz="0 0 0" rpy="0  1.57 0"/>
+    		</xacro:robotiq_85_gripper>
 		<!--Define the position of the TCP with respect to the arm flange-->
 		<joint name="arm_right_tool0_to_tcp" type="fixed" >
@@ -43,6 +41,11 @@
 			<parent link="${prefix}arm_left_link_tool0" />
 			<child link = "${prefix}arm_left_tcp_link" />
-			<origin xyz="0 0 -0.15" rpy="3.1416 0 0.7854" />
+			<origin xyz="0 0 -0.13" rpy="3.1416 0 1.5708" />
 		</joint>
-		</xacro:macro>
+     </xacro:macro>
+<!-- The following xacro is kept for backwards compatibility, it should not be used -->
+<!-- see: https://github.com/ros-industrial/motoman/issues/166 -->
+     <!--xacro:macro name="sda10f">
+          <xacro:motoman_sda10f prefix=""/>
+     </xacro:macro-->
 </robot>

File: motoman_sda10f_support/urdf/simple_sda10f.xacro (robot description, xacro)
@@ -1,5 +1,5 @@
 <?xml version="1.0" ?>
 <robot name="motoman_sda10f" xmlns:xacro="http://ros.org/wiki/xacro">
-	<xacro:include filename="$(find motoman_sda10f_support)/urdf/simple_sda10f_macro.xacro" />
+	<xacro:include filename="$(find motoman_sda10f_support)/urdf/sda10f_macro.xacro" /> <!--version original simple_sda10f_macro.xacro-->
 	<xacro:motoman_sda10f prefix=""/>
 </robot>
