Commit message: s gripper added

File: motoman_sda10f_support/urdf/sda10f_macro.xacro (robot description, xacro)
@@ -5,5 +5,5 @@
      <xacro:include filename="$(find motoman_sda10f_support)/urdf/aruco_marker_macro.xacro"/>
      <xacro:include filename="$(find robotiq_c2_model_visualization)/urdf/robotiq_c2_model_macro.xacro"/>
-     <!--xacro:include filename="$(find robotiq_s_model_visualization)/cfg/s-model_articulated_macro.xacro"/-->
+     <xacro:include filename="$(find robotiq_s_model_visualization)/cfg/s-model_articulated_macro.xacro"/>
      <xacro:include filename="$(find motoman_sda10f_support)/urdf/kinect_macro.xacro" />
 	<xacro:include filename="$(find motoman_sda10f_support)/urdf/environment_macro.xacro"/>
@@ -18,5 +18,5 @@
         </xacro:motoman_arm>
         <xacro:robotiq_c2_model prefix=""/>
-        <!--xacro:s-model_articulated prefix=""/-->
+        <xacro:s-model_articulated prefix=""/>
         	<joint name="left_gripper_to_robot" type="fixed">
 			<parent link="${prefix}arm_left_link_tool0" />
@@ -24,9 +24,9 @@
 			<origin xyz="0 0 0" rpy="0 1.5708 2.3562" />
 		</joint>
-        	<!--joint name="right_gripper_to_robot" type="fixed">
+        	<joint name="right_gripper_to_robot" type="fixed">
 			<parent link="${prefix}arm_right_link_tool0" />
 			<child link = "${prefix}palm" />
 			<origin xyz="0 0 0" rpy="-1.5708 0 1.5708" />
-		</joint-->
+		</joint>
 	  <xacro:aruco_marker prefix=""/>
      </xacro:macro>

Commit message: TCPs added

File: motoman_sda10f_support/urdf/sda10f_macro.xacro (robot description, xacro)
@@ -1,36 +1,47 @@
 <?xml version="1.0" ?>
 <robot xmlns:xacro="http://ros.org/wiki/xacro">
-     <xacro:include filename="$(find motoman_sda10f_support)/urdf/common_torso_macro.xacro" />
-     <xacro:include filename="$(find motoman_sda10f_support)/urdf/arm_macro.xacro" />
-     <xacro:include filename="$(find robotiq_c2_model_visualization)/urdf/robotiq_c2_model_macro.xacro"/>
-     <xacro:include filename="$(find robotiq_s_model_visualization)/cfg/s-model_articulated_macro.xacro"/>
-     <xacro:include filename="$(find motoman_sda10f_support)/urdf/kinect_macro.xacro" />
+	<xacro:include filename="$(find motoman_sda10f_support)/urdf/common_torso_macro.xacro" />
+	<xacro:include filename="$(find motoman_sda10f_support)/urdf/arm_macro.xacro" />
+	<xacro:include filename="$(find robotiq_c2_model_visualization)/urdf/robotiq_c2_model_macro.xacro"/>
+	<xacro:include filename="$(find robotiq_s_model_visualization)/cfg/s-model_articulated_macro.xacro"/>
+	<xacro:include filename="$(find motoman_sda10f_support)/urdf/kinect_macro.xacro" />
 	<xacro:include filename="$(find motoman_sda10f_support)/urdf/environment_macro.xacro"/>
 	<xacro:include filename="$(find motoman_sda10f_support)/urdf/visual_environment_macro.xacro"/>
-     <xacro:macro name="motoman_sda10f" params="prefix">
-        <xacro:torso name="${prefix}torso" prefix="${prefix}torso_"/>
-        <xacro:motoman_arm name="${prefix}arm_left" prefix="${prefix}arm_left_" parent="${prefix}torso_link_b1" reflect="1">
-            <origin xyz="0.09996 0.0275 0.32214" rpy="1.57 0 0" />
-        </xacro:motoman_arm>
-        <xacro:motoman_arm name="${prefix}arm_right" prefix="${prefix}arm_right_" parent="${prefix}torso_link_b1" reflect="-1">
-            <origin xyz="0.09996 -0.0275 0.32214" rpy="1.57 0 0" />
-        </xacro:motoman_arm>
-        <xacro:robotiq_c2_model prefix=""/>
-        <xacro:s-model_articulated prefix=""/>
-        	<joint name="left_gripper_to_robot" type="fixed">
+		<xacro:macro name="motoman_sda10f" params="prefix">
+		<xacro:torso name="${prefix}torso" prefix="${prefix}torso_"/>
+		<xacro:motoman_arm name="${prefix}arm_left" prefix="${prefix}arm_left_" parent="${prefix}torso_link_b1" reflect="1">
+			<origin xyz="0.09996 0.0275 0.32214" rpy="1.57 0 0" />
+		</xacro:motoman_arm>
+		<xacro:motoman_arm name="${prefix}arm_right" prefix="${prefix}arm_right_" parent="${prefix}torso_link_b1" reflect="-1">
+			<origin xyz="0.09996 -0.0275 0.32214" rpy="1.57 0 0" />
+		</xacro:motoman_arm>
+		<!--Grippers-->
+		<xacro:robotiq_c2_model prefix=""/>
+		<xacro:s-model_articulated prefix=""/>
+		<!--Grippers with robotr joints-->
+		<joint name="left_gripper_to_robot" type="fixed">
 			<parent link="${prefix}arm_left_link_tool0" />
 			<child link = "${prefix}robotiq_85_adapter_link" />
 			<origin xyz="0 0 0" rpy="0 1.5708 2.3562" />
 		</joint>
-        	<joint name="right_gripper_to_robot" type="fixed">
+		<joint name="right_gripper_to_robot" type="fixed">
 			<parent link="${prefix}arm_right_link_tool0" />
 			<child link = "${prefix}palm" />
 			<origin xyz="0 0 0" rpy="-1.5708 0 1.5708" />
 		</joint>
-     </xacro:macro>
-<!-- The following xacro is kept for backwards compatibility, it should not be used -->
-<!-- see: https://github.com/ros-industrial/motoman/issues/166 -->
-     <!--xacro:macro name="sda10f">
-          <xacro:motoman_sda10f prefix=""/>
-     </xacro:macro-->
+		<!--Create and update TCP pose -->
+		<link name="arm_right_tcp_link" />
+		<link name="arm_left_tcp_link" />
+		<!--Define the position of the TCP with respect to the arm flange-->
+		<joint name="arm_right_tool0_to_tcp" type="fixed" >
+			<parent link="${prefix}arm_right_link_tool0" />
+			<child link = "${prefix}arm_right_tcp_link" />
+			<origin xyz="0 0 -0.16" rpy="3.1416 0 0" />
+		</joint>
+		<joint name="arm_left_tool0_to_tcp" type="fixed" >
+			<parent link="${prefix}arm_left_link_tool0" />
+			<child link = "${prefix}arm_left_tcp_link" />
+			<origin xyz="0 0 -0.12" rpy="3.1416 0 0.7854" />
+		</joint>
+		</xacro:macro>
 </robot>

Commit message: Right gripper TCP correction

File: motoman_sda10f_support/urdf/sda10f_macro.xacro (robot description, xacro)
@@ -38,5 +38,5 @@
 			<parent link="${prefix}arm_right_link_tool0" />
 			<child link = "${prefix}arm_right_tcp_link" />
-			<origin xyz="0 0 -0.23" rpy="3.1416 0 0" />
+			<origin xyz="0 0 -0.23" rpy="3.1416 0 1.5708" />
 		</joint>
 		<joint name="arm_left_tool0_to_tcp" type="fixed" >

File: motoman_sda10f_support/urdf/simple_sda10f_macro.xacro (robot description, xacro)
@@ -37,5 +37,5 @@
 			<parent link="${prefix}arm_right_link_tool0" />
 			<child link = "${prefix}arm_right_tcp_link" />
-			<origin xyz="0 0 -0.23" rpy="3.1416 0 0" />
+			<origin xyz="0 0 -0.23" rpy="3.1416 0 1.5708" />
 		</joint>
 		<joint name="arm_left_tool0_to_tcp" type="fixed" >

Commit message: tcp update

File: motoman_sda10f_support/urdf/sda10f_macro.xacro (robot description, xacro)
@@ -39,5 +39,5 @@
 			<parent link="${prefix}arm_left_link_tool0" />
 			<child link = "${prefix}arm_left_tcp_link" />
-			<origin xyz="0 0 -0.13" rpy="3.1416 0 1.5708" />
+			<origin xyz="0 0 -0.11" rpy="3.1416 0 1.5708" />
 		</joint>
      </xacro:macro>
