Commit message: URDF update

File: motoman_sda10f_support/urdf/sda10f.xacro (robot description, xacro)
@@ -1,5 +1,5 @@
 <?xml version="1.0" ?>
 <robot name="motoman_sda10f" xmlns:xacro="http://ros.org/wiki/xacro">
-	<xacro:include filename="$(find motoman_sda10f_support)/urdf/simple_sda10f_macro.xacro" /><!--OJO DEVOLVER A LA VERSION ORIGINAL-->
+	<xacro:include filename="$(find motoman_sda10f_support)/urdf/sda10f_macro.xacro" />
 	<xacro:motoman_sda10f prefix=""/>
 </robot>

File: motoman_sda10f_support/urdf/sda10f_macro.xacro (robot description, xacro)
@@ -1,11 +1,16 @@
 <?xml version="1.0" ?>
 <robot xmlns:xacro="http://ros.org/wiki/xacro">
-     <xacro:include filename="$(find motoman_sda10f_support)/urdf/common_torso_macro.xacro" />
-     <xacro:include filename="$(find motoman_sda10f_support)/urdf/arm_macro.xacro" />
-     <xacro:include filename="$(find robotiq_s_model_visualization)/cfg/s-model_articulated_macro.xacro"/>
-     <xacro:include filename="$(find motoman_sda10f_support)/urdf/kinect_macro.xacro" />
-	<xacro:include filename="$(find motoman_sda10f_support)/urdf/environment_macro.xacro"/>
-	<xacro:include filename="$(find motoman_sda10f_support)/urdf/real_sense_macro.xacro"/>
-	<xacro:include filename="$(find robotiq_85_description)/urdf/robotiq_85_gripper.xacro" />
+	<!-- Robot include-->
+     <xacro:include filename="$(find motoman_sda10f_support)/urdf/lenny/common_torso_macro.xacro" />
+     <xacro:include filename="$(find motoman_sda10f_support)/urdf/lenny/arm_macro.xacro" />
+     <!-- Grippers include-->
+     <xacro:include filename="$(find robotiq_2f_85_gripper_visualization)/urdf/robotiq_arg2f_85_model.xacro"/>
+     <xacro:include filename="$(find robotiq_3f_gripper_visualization)/cfg/robotiq-3f-gripper_articulated.xacro"/>
+     <!-- Cameras include-->
+     <xacro:include filename="$(find motoman_sda10f_support)/urdf/cameras/cameras_macro.xacro" />
+     <!-- Environment include-->
+	<xacro:include filename="$(find motoman_sda10f_support)/urdf/environment/environment_macro.xacro"/>
+	<xacro:include filename="$(find motoman_sda10f_support)/urdf/environment/visual_environment_macro.xacro"/>
+	<!--xacro:include filename="$(find motoman_sda10f_support)/urdf/environment/aruco_marker_macro.xacro"/<!-Used for camera calibration ONLY-->
      <xacro:macro name="motoman_sda10f" params="prefix">
         <xacro:torso name="${prefix}torso" prefix="${prefix}torso_"/>
@@ -16,7 +21,10 @@
             <origin xyz="0.09996 -0.0275 0.32214" rpy="1.57 0 0" />
         </xacro:motoman_arm>
-        <!--xacro:robotiq_c2_model prefix=""/-->
-		<xacro:s-model_articulated prefix=""/>
-		<!--Grippers with robot joints-->
+        <!--Grippers with robot joints-->
+		<joint name="left_gripper_to_robot" type="fixed">
+			<parent link="${prefix}arm_left_link_tool0" />
+			<child link = "${prefix}robotiq_arg2f_base_link" />
+			<origin xyz="0 0 0" rpy="0 3.1416 -0.7854" />
+		</joint>
 		<joint name="right_gripper_to_robot" type="fixed">
 			<parent link="${prefix}arm_right_link_tool0" />
@@ -27,7 +35,4 @@
 		<link name="arm_right_tcp_link" />
 		<link name="arm_left_tcp_link" />
-		<xacro:robotiq_85_gripper prefix="" parent="arm_left_link_tool0" >
-        		<origin xyz="0 0 0" rpy="0  1.57 0"/>
-    		</xacro:robotiq_85_gripper>
 		<!--Define the position of the TCP with respect to the arm flange-->
 		<joint name="arm_right_tool0_to_tcp" type="fixed" >
@@ -39,5 +44,5 @@
 			<parent link="${prefix}arm_left_link_tool0" />
 			<child link = "${prefix}arm_left_tcp_link" />
-			<origin xyz="0 0 -0.11" rpy="3.1416 0 1.5708" />
+			<origin xyz="0 0 -0.15" rpy="3.1416 0 0.7854" />
 		</joint>
      </xacro:macro>
