Commit message: Environment refurbished

File: motoman_sda10f_support/urdf/cameras/kinect_macro.xacro (robot description, xacro)
@@ -59,26 +59,4 @@
 		</visual>
 	</link>
-		<!-- joint list -->
-	<joint name="base_kinect_to_robot" type="fixed"> <!--ACTUALIZAR CON DATA REAL OJO MODIFICAR AQUI-->
-		<parent link="torso_base_link"/>
-		<child link="base_kinect"/>
-		<origin xyz="0.817 0.056 2.07" rpy="1.5708 0 -1.52"/> <!--origin xyz="0.148 0.845 1.6425" rpy="1.54 0 -3.14"/> <ESTA ES LA TRANSFORMADA QUE HAY QUE MEDIR menos 30cm en Z-->
-	</joint>
-	<joint name="base_kinect2_to_robot" type="fixed">
-		<parent link="torso_base_link"/>
-		<child link="base_kinect2"/>
-		<origin xyz="0.9 -3 1.8" rpy="0.2443 0 3.1416"/>
-	</joint>
-	<joint name="base_kinect_to_kinect" type="fixed">
-		<parent link="base_kinect"/>
-		<child link="kinect"/>
-		<origin xyz="0 0 0" rpy="0 0 0"/>
-	</joint>
-	<joint name="base_kinect2_to_kinect2" type="fixed">
-		<parent link="base_kinect2"/>
-		<child link="kinect2"/>
-		<origin xyz="0 0 0" rpy="0 0 0"/>
-	</joint>
-		<!-- end of joint list -->
 	</xacro:macro>
 	<xacro:kinect name="kinect" prefix="kinect_"/>

File: motoman_sda10f_support/urdf/cameras/zed_macro.xacro (robot description, xacro)
@@ -56,3 +56,4 @@
     <link name="zed_right_camera_optical_frame"/>
     </xacro:macro>
+    <xacro:zed_camera prefix=""/>
 </robot>

File: motoman_sda10f_support/urdf/environment/environment_macro.xacro (robot description, xacro)
@@ -1,7 +1,5 @@
 <?xml version="1.0" ?>
 <model xmlns:xacro="http://ros.org/wiki/xacro">
-	<xacro:include filename="$(find motoman_sda10f_support)/urdf/zed_macro.xacro"/><!-- ZED camera -->
 	<xacro:macro name="environment" params="name prefix">
-	<xacro:zed_camera prefix=""/>
 		<!-- link list -->
 	<link name="conveyor">
@@ -74,6 +72,6 @@
 			</geometry>
 			<origin xyz="0 0 0"/>
-			<material name="gray_conveyor">
-				<texture filename="package://motoman_sda10f_support/meshes/environment/textures/red.png"/>
+			<material name="gray_worktable">
+				<color rgba="${45/255} ${135/255} ${149/255} 1"/>
 			</material>
 		</visual>
@@ -197,10 +195,4 @@
 		<origin xyz="-1.35 0.6 -0.3" rpy="0 0 -1.5708"/> <!Sumo 5cm a las MPS por si acaso-->
 	<!--/joint-->
-	<!-- Camera zed -->
-	<joint name="zed_camera" type="fixed">
-		<parent link="torso_base_link" />
-		<child link = "zed_camera_center" />
-		<origin xyz="0.8 0.05 2.05" rpy="0 1.57 0" />
-	</joint>
 	<joint name="tooltable_to_robot" type="fixed">
 		<parent link="conveyor"/>

File: motoman_sda10f_support/urdf/sda10f.xacro (robot description, xacro)
@@ -1,5 +1,5 @@
 <?xml version="1.0" ?>
 <robot name="motoman_sda10f" xmlns:xacro="http://ros.org/wiki/xacro">
-	<xacro:include filename="$(find motoman_sda10f_support)/urdf/sda10f_macro.xacro" />
+	<xacro:include filename="$(find motoman_sda10f_support)/urdf/simple_sda10f_macro.xacro" /><!--OJO DEVOLVER A LA VERSION ORIGINAL-->
 	<xacro:motoman_sda10f prefix=""/>
 </robot>

File: motoman_sda10f_support/urdf/simple_sda10f.xacro (robot description, xacro)
@@ -1,5 +1,5 @@
 <?xml version="1.0" ?>
 <robot name="motoman_sda10f" xmlns:xacro="http://ros.org/wiki/xacro">
-	<xacro:include filename="$(find motoman_sda10f_support)/urdf/sda10f_macro.xacro" /> <!--version original simple_sda10f_macro.xacro-->
+	<xacro:include filename="$(find motoman_sda10f_support)/urdf/simple_sda10f_macro.xacro"/>
 	<xacro:motoman_sda10f prefix=""/>
 </robot>

File: motoman_sda10f_support/urdf/simple_sda10f_macro.xacro (robot description, xacro)
@@ -1,11 +1,15 @@
 <?xml version="1.0" ?>
 <robot xmlns:xacro="http://ros.org/wiki/xacro">
-     <xacro:include filename="$(find motoman_sda10f_support)/urdf/common_torso_macro.xacro" />
-     <xacro:include filename="$(find motoman_sda10f_support)/urdf/arm_macro.xacro" />
-     <xacro:include filename="$(find robotiq_s_model_visualization)/cfg/s-model_articulated_macro.xacro"/>
-     <xacro:include filename="$(find motoman_sda10f_support)/urdf/kinect_macro.xacro" />
-	<xacro:include filename="$(find motoman_sda10f_support)/urdf/environment_macro.xacro"/>
-	<xacro:include filename="$(find motoman_sda10f_support)/urdf/real_sense_macro.xacro"/>
-	<xacro:include filename="$(find robotiq_85_description)/urdf/robotiq_85_gripper.xacro" />
+	<!-- Robot include-->
+     <xacro:include filename="$(find motoman_sda10f_support)/urdf/lenny/common_torso_macro.xacro" />
+     <xacro:include filename="$(find motoman_sda10f_support)/urdf/lenny/arm_macro.xacro" />
+     <!-- Grippers include-->
+     <xacro:include filename="$(find robotiq_2f_85_gripper_visualization)/urdf/robotiq_arg2f_85_model.xacro"/>
+     <xacro:include filename="$(find robotiq_3f_gripper_visualization)/cfg/robotiq-3f-gripper_articulated.xacro"/>
+     <!-- Cameras include-->
+     <xacro:include filename="$(find motoman_sda10f_support)/urdf/cameras/cameras_macro.xacro" />
+     <!-- Environment include-->
+	<xacro:include filename="$(find motoman_sda10f_support)/urdf/environment/environment_macro.xacro"/>
+	<!--xacro:include filename="$(find motoman_sda10f_support)/urdf/environment/aruco_marker_macro.xacro"/<!-Used for camera calibration ONLY-->
      <xacro:macro name="motoman_sda10f" params="prefix">
         <xacro:torso name="${prefix}torso" prefix="${prefix}torso_"/>
@@ -16,7 +20,10 @@
             <origin xyz="0.09996 -0.0275 0.32214" rpy="1.57 0 0" />
         </xacro:motoman_arm>
-        <!--xacro:robotiq_c2_model prefix=""/-->
-		<xacro:s-model_articulated prefix=""/>
-		<!--Grippers with robot joints-->
+        <!--Grippers with robot joints-->
+		<joint name="left_gripper_to_robot" type="fixed">
+			<parent link="${prefix}arm_left_link_tool0" />
+			<child link = "${prefix}robotiq_arg2f_base_link" />
+			<origin xyz="0 0 0" rpy="0 3.1416 -0.7854" />
+		</joint>
 		<joint name="right_gripper_to_robot" type="fixed">
 			<parent link="${prefix}arm_right_link_tool0" />
@@ -27,7 +34,4 @@
 		<link name="arm_right_tcp_link" />
 		<link name="arm_left_tcp_link" />
-		<xacro:robotiq_85_gripper prefix="" parent="arm_left_link_tool0" >
-        		<origin xyz="0 0 0" rpy="0  1.57 0"/>
-    		</xacro:robotiq_85_gripper>
 		<!--Define the position of the TCP with respect to the arm flange-->
 		<joint name="arm_right_tool0_to_tcp" type="fixed" >
@@ -39,5 +43,5 @@
 			<parent link="${prefix}arm_left_link_tool0" />
 			<child link = "${prefix}arm_left_tcp_link" />
-			<origin xyz="0 0 -0.13" rpy="3.1416 0 1.5708" />
+			<origin xyz="0 0 -0.15" rpy="3.1416 0 0.7854" />
 		</joint>
      </xacro:macro>
